File: Sesion2_Izan/Alimentacion.kicad_sch (KiCad schematic)
At the start: 0 parts

Commit message: Complete power supply schematic
Parts:
- added C1: 100nF, Capacitor_SMD:C_0805_2012Metric_Pad1.18x1.45mm_HandSolder, symbol Device:C
- added C2: 10uF, Capacitor_Tantalum_SMD:CP_EIA-3216-18_Kemet-A, symbol Device:C_Polarized
- added U1: LD1117S33TR_SOT223, Package_TO_SOT_SMD:SOT-223-3_TabPin2, symbol Regulator_Linear:LD1117S33TR_SOT223
Connections:
- new net 3V3: C2.1, U1.2 (VO)
- new net GND: C1.2, C2.2, U1.1 (GND)
- new net VIN: C1.1, U1.3 (VI)

Commit message: Complete microcontroller schematic and BOM
Parts:
- renumbered C1 to C201, C2 to C202, U1 to U201
Changed lines of the file:
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@@
 		(dnp no)
 		(fields_autoplaced yes)
-		(property "Reference" "#PWR02"
+		(property "Reference" "#PWR0202"
 			(at 138.43 121.92 0)
 			(hide yes)
@@
 			(project "Sesion2_Izan"
 				(path "/e349a083-9e3b-40e5-ab26-55c4e44866b1/67a69597-7fdb-464d-b33e-0e119b3f6ebb"
-					(reference "#PWR02")
+					(reference "#PWR0202")
 					(unit 1)
 				)
@@
 		(dnp no)
 		(fields_autoplaced yes)
-		(property "Reference" "U1"
+		(property "Reference" "U201"
 			(at 138.43 93.98 0)
 			(show_name no)
@@
 			(project "Sesion2_Izan"
 				(path "/e349a083-9e3b-40e5-ab26-55c4e44866b1/67a69597-7fdb-464d-b33e-0e119b3f6ebb"
-					(reference "U1")
+					(reference "U201")
 					(unit 1)
 				)
@@
 		(dnp no)
 		(fields_autoplaced yes)
-		(property "Reference" "#PWR01"
+		(property "Reference" "#PWR0201"
 			(at 121.92 121.92 0)
 			(hide yes)
@@
 			(project "Sesion2_Izan"
 				(path "/e349a083-9e3b-40e5-ab26-55c4e44866b1/67a69597-7fdb-464d-b33e-0e119b3f6ebb"
-					(reference "#PWR01")
+					(reference "#PWR0201")
 					(unit 1)
 				)
@@
 		(dnp no)
 		(fields_autoplaced yes)
-		(property "Reference" "C2"
+		(property "Reference" "C202"
 			(at 157.48 105.7909 0)
 			(show_name no)
@@
 			(project "Sesion2_Izan"
 				(path "/e349a083-9e3b-40e5-ab26-55c4e44866b1/67a69597-7fdb-464d-b33e-0e119b3f6ebb"
-					(reference "C2")
+					(reference "C202")
 					(unit 1)
 				)
@@
 		(dnp no)
 		(fields_autoplaced yes)
-		(property "Reference" "#PWR03"
+		(property "Reference" "#PWR0203"
 			(at 153.67 121.92 0)
 			(hide yes)
@@
 			(project "Sesion2_Izan"
 				(path "/e349a083-9e3b-40e5-ab26-55c4e44866b1/67a69597-7fdb-464d-b33e-0e119b3f6ebb"
-					(reference "#PWR03")
+					(reference "#PWR0203")
 					(unit 1)
 				)
@@
 		(dnp no)
 		(fields_autoplaced yes)
-		(property "Reference" "C1"
+		(property "Reference" "C201"
 			(at 125.73 106.6799 0)
 			(show_name no)
@@
 			(project "Sesion2_Izan"
 				(path "/e349a083-9e3b-40e5-ab26-55c4e44866b1/67a69597-7fdb-464d-b33e-0e119b3f6ebb"
-					(reference "C1")
+					(reference "C201")
 					(unit 1)
 				)
