File: Sesion2_Izan/Alimentacion.kicad_sch (KiCad schematic)
At the start: 3 parts, among them U201 LD1117S33TR_SOT223

Commit message: S3: add MCU decoupling and power test points
Schematic changes for Session 3, based on the component datasheets:
- C302 100nF + C303 4.7uF (X7R, 0805) on U301 VDD/VDDA (pin 4), as
  required by the STM32G030 power supply scheme (DS12991, Figure 9)
- TP201 VIN, TP202 3V3 and TP203 GND test points (Keystone 5003/5000/5001)
- LD1117 input/output capacitors (C201 100nF, C202 10uF tantalum) already
  match the LD1117 application circuit; NRST already has C301 100nF
- BOM regenerated with the S2 column set (19 components)
- ERC: 0 errors, 0 warnings (S3_validation/ERC_report.*)

Co-Authored-By: Claude Opus 5.5 <noreply@anthropic.com>
Parts:
- added TP201: VIN, TestPoint:TestPoint_Keystone_5000-5004_Miniature, symbol Connector:TestPoint
- added TP202: 3V3, TestPoint:TestPoint_Keystone_5000-5004_Miniature, symbol Connector:TestPoint
- added TP203: GND, TestPoint:TestPoint_Keystone_5000-5004_Miniature, symbol Connector:TestPoint
Connections:
- net 3V3: now also TP202.1
- net GND: now also TP203.1
- net VIN: now also TP201.1
