File: Sesion2_Izan/Microcontrolador.kicad_sch (KiCad schematic)
At the start: 0 parts

Commit message: Complete microcontroller schematic and BOM
Parts:
- added C301: 100 nF, Capacitor_SMD:C_0805_2012Metric_Pad1.18x1.45mm_HandSolder, symbol Device:C
- added J301: E/S, Connector_PinHeader_2.54mm:PinHeader_1x06_P2.54mm_Vertical, symbol Connector_Generic:Conn_01x06
- added J302: SWD, Connector_PinHeader_2.54mm:PinHeader_1x05_P2.54mm_Vertical, symbol Connector_Generic:Conn_01x05
- added U301: STM32G030K8Tx, Package_QFP:LQFP-32_7x7mm_P0.8mm, symbol MCU_ST_STM32G0:STM32G030K8Tx
Connections:
- new net 3V3: J301.1 (Pin_1), J302.1 (Pin_1), U301.4 (VDD)
- new net AIN1: U301.7 (PA0)
- new net AIN1_EXT: J301.2 (Pin_2)
- new net AIN2: U301.8 (PA1)
- new net AIN2_EXT: J301.3 (Pin_3)
- new net AIN3: U301.11 (PA4)
- new net AIN3_EXT: J301.4 (Pin_4)
- new net GND: C301.2, J301.6 (Pin_6), J302.3 (Pin_3), U301.5 (VSS)
- new net NRST: C301.1, J302.5 (Pin_5), U301.6 (NRST)
- new net OUT1: J301.5 (Pin_5), U301.12 (PA5)
- new net SWCLK: J302.2 (Pin_2), U301.25 (PA14)
- new net SWDIO: J302.4 (Pin_4), U301.24 (PA13)
- no-connect marks 0 -> 21
Other:
- added sheet FiltroRC_1 (FiltroRC.kicad_sch)
- added sheet FiltroRC_2 (FiltroRC.kicad_sch)
- added sheet FiltroRC_3 (FiltroRC.kicad_sch)
