File: Sesion2_Izan/Microcontrolador.kicad_sch (KiCad schematic)
At the start: 4 parts, among them J301 E/S, J302 SWD, U301 STM32G030K8Tx

Commit message: S3: carry over pending KiCad edits found uncommitted on main
These edits were in the working tree when Session 3 started (KiCad
local history: "SCH Save" 2026-10-01 02:50, after S2 commit 9509303).
They are committed here, on the S3 branch, so main stays untouched:

- BOM export settings: Manufacturer and MPN columns, export filename
- C301 value normalized from "100 nF" to "100nF"
- FiltroRC.kicad_sch sheet UUID regenerated by KiCad on save

Co-Authored-By: Claude Opus 5.5 <noreply@anthropic.com>
Parts:
- C301: value 100 nF -> 100nF
Changed lines of the file:
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@@
 			)
 		)
-		(property "Value" "100 nF"
+		(property "Value" "100nF"
 			(at 109.22 59.69 90)
 			(show_name no)

Commit message: S3: add MCU decoupling and power test points
Schematic changes for Session 3, based on the component datasheets:
- C302 100nF + C303 4.7uF (X7R, 0805) on U301 VDD/VDDA (pin 4), as
  required by the STM32G030 power supply scheme (DS12991, Figure 9)
- TP201 VIN, TP202 3V3 and TP203 GND test points (Keystone 5003/5000/5001)
- LD1117 input/output capacitors (C201 100nF, C202 10uF tantalum) already
  match the LD1117 application circuit; NRST already has C301 100nF
- BOM regenerated with the S2 column set (19 components)
- ERC: 0 errors, 0 warnings (S3_validation/ERC_report.*)

Co-Authored-By: Claude Opus 5.5 <noreply@anthropic.com>
Parts:
- added C302: 100nF, Capacitor_SMD:C_0805_2012Metric_Pad1.18x1.45mm_HandSolder, symbol Device:C
- added C303: 4.7uF, Capacitor_SMD:C_0805_2012Metric_Pad1.18x1.45mm_HandSolder, symbol Device:C
Connections:
- net 3V3: now also C302.1, C303.1
- net GND: now also C302.2, C303.2
